Commit message: Renamed Project

File: trail_patrol_drone/urdf/husky.gazebo.xacro (robot description, xacro)
@@ -4,5 +4,5 @@
   <xacro:arg name="camera_visual" default="false"/>
   <xacro:arg name="imu_visual"    default="false"/>
-  <xacro:include filename="$(find 41068_ignition_bringup)/urdf/wheel.urdf.xacro"/>
+  <xacro:include filename="$(find trail_patrol_drone)/urdf/wheel.urdf.xacro"/>
   <gazebo reference="imu_link">
     <sensor type="imu" name="imu">

File: trail_patrol_drone/urdf/husky.urdf.xacro (robot description, xacro)
@@ -1,7 +1,7 @@
 <?xml version="1.0" ?>
 <robot name="husky" xmlns:xacro="http://ros.org/wiki/xacro">
-  <xacro:include filename="$(find 41068_ignition_bringup)/urdf/common_properties.urdf.xacro"/>
-  <xacro:include filename="$(find 41068_ignition_bringup)/urdf/husky.gazebo.xacro"/>
-  <xacro:include filename="$(find 41068_ignition_bringup)/urdf/wheel.urdf.xacro"/>
+  <xacro:include filename="$(find trail_patrol_drone)/urdf/common_properties.urdf.xacro"/>
+  <xacro:include filename="$(find trail_patrol_drone)/urdf/husky.gazebo.xacro"/>
+  <xacro:include filename="$(find trail_patrol_drone)/urdf/wheel.urdf.xacro"/>
   <xacro:property name="r200_cam_rgb_px" value="0.005"/>
   <xacro:property name="r200_cam_rgb_py" value="0.018"/>
@@ -12,5 +12,5 @@
       <origin xyz="0 0 0.0" rpy="0 0 0"/>
       <geometry>
-        <mesh filename="file://$(find 41068_ignition_bringup)/urdf/meshes/base_link.dae"/>
+        <mesh filename="file://$(find trail_patrol_drone)/urdf/meshes/base_link.dae"/>
       </geometry>
       <material name="black"/>
@@ -19,5 +19,5 @@
       <origin xyz="0.48 0 0.091" rpy="0 0 0"/>
       <geometry>
-        <mesh filename="file://$(find 41068_ignition_bringup)/urdf/meshes/bumper.dae"/>
+        <mesh filename="file://$(find trail_patrol_drone)/urdf/meshes/bumper.dae"/>
       </geometry>
       <material name="black"/>
@@ -26,5 +26,5 @@
       <origin xyz="-0.48 0 0.091" rpy="0 0 3.14159"/>
       <geometry>
-        <mesh filename="file://$(find 41068_ignition_bringup)/urdf/meshes/bumper.dae"/>
+        <mesh filename="file://$(find trail_patrol_drone)/urdf/meshes/bumper.dae"/>
       </geometry>
       <material name="black"/>
@@ -33,5 +33,5 @@
       <origin xyz="0 0 0" rpy="0 0 0"/>
       <geometry>
-        <mesh filename="file://$(find 41068_ignition_bringup)/urdf/meshes/top_chassis.dae"/>
+        <mesh filename="file://$(find trail_patrol_drone)/urdf/meshes/top_chassis.dae"/>
       </geometry>
     </visual>
@@ -39,5 +39,5 @@
       <origin xyz="0.0812 0 0.245" rpy="0 0 0"/>
       <geometry>
-        <mesh filename="file://$(find 41068_ignition_bringup)/urdf/meshes/top_plate.dae"/>
+        <mesh filename="file://$(find trail_patrol_drone)/urdf/meshes/top_plate.dae"/>
       </geometry>
       <material name="black"/>
@@ -46,5 +46,5 @@
       <origin xyz="0.0012 0 0.251" rpy="0 0 0"/>
       <geometry>
-        <mesh filename="file://$(find 41068_ignition_bringup)/urdf/meshes/jpl04_arch_nosensor.stl"/>
+        <mesh filename="file://$(find trail_patrol_drone)/urdf/meshes/jpl04_arch_nosensor.stl"/>
       </geometry>
       <material name="black"/>
@@ -71,5 +71,5 @@
       <origin xyz="0.0812 0 0.245" rpy="0 0 0"/>
       <geometry>
-        <mesh filename="file://$(find 41068_ignition_bringup)/urdf/meshes/top_plate.dae"/>
+        <mesh filename="file://$(find trail_patrol_drone)/urdf/meshes/top_plate.dae"/>
       </geometry>
     </collision>

File: trail_patrol_drone/urdf/wheel.urdf.xacro (robot description, xacro)
@@ -9,5 +9,5 @@
         <origin xyz="0 0 0" rpy="0 0 0"/>
         <geometry>
-          <mesh filename="file://$(find 41068_ignition_bringup)/urdf/meshes/wheel.dae"/>
+          <mesh filename="file://$(find trail_patrol_drone)/urdf/meshes/wheel.dae"/>
         </geometry>
       </visual>

File: trail_patrol_drone/urdf_drone/parrot.gazebo.xacro (robot description, xacro)
@@ -4,5 +4,5 @@
   <xacro:arg name="camera_visual" default="false"/>
   <xacro:arg name="imu_visual"    default="false"/>
-  <!-- <xacro:include filename="$(find 41068_ignition_bringup)/urdf/wheel.urdf.xacro"/> -->
+  <!-- <xacro:include filename="$(find trail_patrol_drone)/urdf/wheel.urdf.xacro"/> -->
   <gazebo reference="imu_link">
     <sensor type="imu" name="imu">

File: trail_patrol_drone/urdf_drone/parrot.urdf.xacro (robot description, xacro)
@@ -1,6 +1,6 @@
 <?xml version="1.0" ?>
 <robot name="parrot" xmlns:xacro="http://ros.org/wiki/xacro">
-  <xacro:include filename="$(find 41068_ignition_bringup)/urdf_drone/common_properties.urdf.xacro"/>
-  <xacro:include filename="$(find 41068_ignition_bringup)/urdf_drone/parrot.gazebo.xacro"/>
+  <xacro:include filename="$(find trail_patrol_drone)/urdf_drone/common_properties.urdf.xacro"/>
+  <xacro:include filename="$(find trail_patrol_drone)/urdf_drone/parrot.gazebo.xacro"/>
   <xacro:property name="r200_cam_rgb_px" value="0.005"/>
   <xacro:property name="r200_cam_rgb_py" value="0.018"/>
@@ -24,5 +24,5 @@
     <visual name="hull">
       <geometry>
-        <mesh filename="file://$(find 41068_ignition_bringup)/urdf_drone/meshes/hull.dae"/>
+        <mesh filename="file://$(find trail_patrol_drone)/urdf_drone/meshes/hull.dae"/>
       </geometry>
     </visual>
@@ -30,5 +30,5 @@
       <origin xyz="-0.09035 -0.11423 -0.00501" rpy="0 0 0"/>
       <geometry>
-        <mesh filename="file://$(find 41068_ignition_bringup)/urdf_drone/meshes/propeller_rr.dae"/>
+        <mesh filename="file://$(find trail_patrol_drone)/urdf_drone/meshes/propeller_rr.dae"/>
       </geometry>
     </visual>
@@ -36,5 +36,5 @@
       <origin xyz="0.09035 0.11452 -0.00501" rpy="0 0 0"/>
       <geometry>
-        <mesh filename="file://$(find 41068_ignition_bringup)/urdf_drone/meshes/propeller_rl.dae"/>
+        <mesh filename="file://$(find trail_patrol_drone)/urdf_drone/meshes/propeller_rl.dae"/>
       </geometry>
     </visual>
@@ -42,5 +42,5 @@
       <origin xyz="0.08456 -0.11435 -0.00501" rpy="0 0 0"/>
       <geometry>
-        <mesh filename="file://$(find 41068_ignition_bringup)/urdf_drone/meshes/propeller_fr.dae"/>
+        <mesh filename="file://$(find trail_patrol_drone)/urdf_drone/meshes/propeller_fr.dae"/>
       </geometry>
     </visual>
@@ -48,5 +48,5 @@
       <origin xyz="0.08456 0.11463 -0.00501" rpy="0 0 0"/>
       <geometry>
-        <mesh filename="file://$(find 41068_ignition_bringup)/urdf_drone/meshes/propeller_fl.dae"/>
+        <mesh filename="file://$(find trail_patrol_drone)/urdf_drone/meshes/propeller_fl.dae"/>
       </geometry>
     </visual>
